Commit message: Task 1.6.1|1.6.2: DH and Inverse Kinematics

File: quadruped_robot/urdf/quadruped_robot.urdf (robot description, URDF)
Before this commit: robot quadruped_robot, 13 links, 12 joints
Links:
- link back_left_leg: mass 6.93816621303876 -> 6.93816847911244
- link back_left_shin: mass 2.18914769812056 -> 2.1890918917642
- link back_left_thigh: mass 0 -> 2.8500353369203
- link back_right_leg: mass 6.93817966820701 -> 6.93816860410077
- link back_right_shin: mass 2.18909743803364 -> 2.18909068675098
- link back_right_thigh: mass 2.85003646130647 -> 2.85003531462536
- link front_left_leg: mass 6.93818133420775 -> 6.93816849077714
- link front_left_shin: mass 2.18909364696934 -> 2.18909081108663
- link front_left_thigh: mass 2.85003544879558 -> 2.8500353343221
- link front_right_leg: mass 6.93816605315389 -> 6.9381686574405
- link front_right_shin: mass 2.18910071138097 -> 2.18909067780491
- link front_right_thigh: mass 2.85 -> 2.85003532279257
Joints:
- joint back_left_leg_joint: axis 1 0 0 -> 0.98197618745736 -0.188099372550818 -0.0184768317818711; origin xyz=0.070172 0 0.081073 rpy=3.0436 -1.5699 -3.1416 -> xyz=0.0701724686163078 0 0.0810726777394658 rpy=3.04358892179118 -1.56986563009081 -3.14159265358249
- joint back_left_shin_joint: axis -1 0 0 -> -0.98197618745736 -0.174417566004741 -0.0728098889965498; origin xyz=0 -0.5 0 rpy=2.8441 0 0 -> xyz=0 -0.5 0 rpy=2.84405277747574 0 0
- joint back_left_thigh_joint: origin xyz=-0.18189 -0.69729 0.59749 rpy=1.362 0 3.1416 -> xyz=-0.249882405181029 0.18 0 rpy=1.36200189468701 0 3.14159265358979
- joint back_right_leg_joint: axis 1 0 0 -> 0.93624 -0.28957 -0.199
- joint back_right_shin_joint: axis -1 0 0 -> -0.93624 -0.31194 0.16169
- joint back_right_thigh_joint: origin xyz=-0.18189 -1.0573 0.59749 rpy=-1.2051 0 3.1416 -> xyz=-0.249882405181029 -0.18 0 rpy=-1.2050955352319 0 3.14159265358979
- joint front_left_leg_joint: axis 1 0 0 -> 0.99608 0.075661 0.045868
- joint front_left_shin_joint: axis -1 0 0 -> -0.996078094500597 -0.0197781632448234 -0.0862395148103312; origin xyz=0.028461 -0.5 0 rpy=-1.8903 0 3.1416 -> xyz=0.028460525371978 -0.5 0 rpy=-1.89034893239217 0 3.14159265358979
- joint front_left_thigh_joint: origin xyz=0.31787 -0.69729 0.59749 rpy=-1.6419 0 0 -> xyz=0.249882405181029 0.18 0 rpy=-1.64194996163522 0 0
- joint front_right_leg_joint: axis 1 0 0 -> 0.96999 -0.23939 0.042598
- joint front_right_shin_joint: axis -1 0 0 -> -0.96999 0.19775 -0.14147
- joint front_right_thigh_joint: origin xyz=0.31787 -1.0573 0.59749 rpy=1.3364 0 0 -> xyz=0.24988 -0.18 0 rpy=1.3364 0 0
