Commit message: Updated Arena

File: field/urdf/field.urdf (robot description, URDF)
Before this commit: robot new_arena, 5 links, 4 joints
Links:
- link arena: geometry collision mesh filename=package://field/meshes/arena.STL; visual mesh filename=package://field/meshes/arena.STL
- link rubble: geometry collision mesh filename=package://field/meshes/rubble.STL; visual mesh filename=package://field/meshes/rubble.STL
- link slope: mass 5300 -> 420; geometry collision mesh filename=package://field/meshes/slope.STL; visual mesh filename=package://field/meshes/slope.STL
- link wall_1: geometry collision mesh filename=package://field/meshes/wall_1.STL; visual mesh filename=package://field/meshes/wall_1.STL
- link wall_2: geometry collision mesh filename=package://field/meshes/wall_2.STL; visual mesh filename=package://field/meshes/wall_2.STL
Joints:
- joint rubble_joint: axis 1 0 0 -> 0 0 0
- joint slope_joint: axis 0 0 0 -> 1 0 0
- joint wall_1_joint: axis 0 0 1 -> 0 0 0
- joint wall_2_joint: axis 0 0 1 -> 1 0 0; origin xyz=3.0334 2.5 0.1 rpy=-1.5708 0 -1.5708 -> xyz=3.03337213258269 2.5 0.0999999999999998 rpy=-1.5707963267949 0 -1.5707963267949
